File: DrawerModeling/DrawerModeling.kicad_sch (KiCad schematic)
At the start: 34 parts, among them SW1 SW_NKK_GW12LJPCF, SW3 SW_SPDT_321, U1 AD633JRZ-R7, U11 TLP222A-2, U2 L7805, U3 LM393_Block, U4 TL082_Block, U6 LM1117LD-3.3, U7 AD633JRZ-R7, U8 L7815, U9 L7915

Commit message: pcb_1
Parts:
- removed C1, C2: 500uF, symbol Device:C_Polarized
- removed C4: 5n, symbol Device:C
- removed D1, D2, D3, D4: D_45deg, symbol Device:D_45deg
- removed RV1: 1000, symbol Device:R_Potentiometer
- removed SW1: SW_NKK_GW12LJPCF, Button_Switch_THT:SW_NKK_GW12LJP, symbol Switch:SW_NKK_GW12LJPCF
- removed SW3: SW_SPDT_321, symbol Switch:SW_SPDT_321
- removed TR1: TEZ4.0-D-2, Transformer_THT:Transformer_Breve_TEZ-35x42, symbol Transformer:TEZ4.0-D-2
- removed U11: TLP222A-2, Package_DIP:DIP-8_W7.62mm, symbol Relay_SolidState:TLP222A-2
- removed U2: L7805, symbol Regulator_Linear:L7805
- removed U3: LM393_Block, Package_DIP:DIP-8_W7.62mm, symbol Ki_Library:LM393_Block
- removed U6: LM1117LD-3.3, Package_SON:WSON-8-1EP_4x4mm_P0.8mm_EP2.2x3mm, symbol Regulator_Linear:LM1117LD-3.3
- removed U7: AD633JRZ-R7, AD633JRZ-R7:SOIC127P600X175-8N, symbol AD633JRZ-R7:AD633JRZ-R7
- removed U8: L7815, symbol Regulator_Linear:L7815
- removed U9: L7915, symbol Regulator_Linear:L7915
- removed V1: VSIN, symbol Simulation_SPICE:VSIN
- added Button1_a1, Button1_a2, Button1_b1, Button1_b2, Button2_a1, Button2_a2, Button2_b1, Button2_b2, ConnView_Modulation1, ConnView_Out1, ConnView_Out2, ConnView_Out3, ConnView_Out4, ConnView_Out5, ConnView_OutInfo1, ConnView_OutLast1: Conn_01x01, Connector_Wire:SolderWirePad_1x01_SMD_1.5x3mm, symbol Connector_Generic:Conn_01x01
- added C1, C10, C13, C14, C5, C6, C7: C, Capacitor_THT:C_Axial_L3.8mm_D2.6mm_P7.50mm_Horizontal, symbol Device:C
- added C4: C_Polarized, Capacitor_THT:CP_Radial_D6.3mm_P2.50mm, symbol Device:C_Polarized
- added C_G1, C_G2: C, Capacitor_SMD:C_0603_1608Metric, symbol Device:C
- added ConnProgramator1: Conn_01x04_Pin, Connector_PinHeader_2.54mm:PinHeader_1x04_P2.54mm_Vertical, symbol Connector:Conn_01x04_Pin
- added D1: D, Diode_SMD:D_MELF-RM10_Universal_Handsoldering, symbol Device:D
- added J1: Conn_01x05_Pin, Connector_PinHeader_2.54mm:PinHeader_1x05_P2.54mm_Vertical, symbol Connector:Conn_01x05_Pin
- added Q1, Q2, Q4, Q5: 2N3904, Package_TO_SOT_THT:TO-92_Inline, symbol Transistor_BJT:2N3904
- added Q3: 2N3906, Package_TO_SOT_THT:TO-92_Inline, symbol Transistor_BJT:2N3906
- added R10, R11, R13, R14, R15, R16, R17, R19, R20, R21, R22, R23, R24, R25, R26, R27, R28, R29, R30, R31, R32, R34, R35, R36, R37, R38, R39, R40, R41, R42, R43, R44, R45, R9: R, Resistor_THT:R_Axial_DIN0207_L6.3mm_D2.5mm_P10.16mm_Horizontal, symbol Device:R
- added R18: R_Potentiometer_US, Potentiometer_THT:Potentiometer_Alps_RK163_Single_Horizontal, symbol Device:R_Potentiometer_US
- added U10, U13, U15, U2, U6, U9: TL072, Package_DIP:DIP-8_W10.16mm, symbol Amplifier_Operational:TL072
- added U11, U12, U16, U17: TLP222A, VikLib:TLP127, symbol Relay_SolidState:TLP222A
- added U14: LM13700, Package_DIP:DIP-16_W7.62mm, symbol Amplifier_Operational:LM13700
- added U18: MCP4725xxx-xCH, Package_TO_SOT_SMD:SOT-23-6, symbol Analog_DAC:MCP4725xxx-xCH
- added U19: XC6206PxxxMR, Package_TO_SOT_SMD:SOT-23-3, symbol Regulator_Linear:XC6206PxxxMR
- added U3: ~, Audio_Module:Arduino_LCD_Shield, symbol MCU_Module:Arduino_LCD_Shield
- added U7: STM32F411CCUx, Package_DFN_QFN:QFN-48-1EP_7x7mm_P0.5mm_EP5.6x5.6mm, symbol MCU_ST_STM32F4:STM32F411CCUx
- added U8: LT1011, Package_SO:SOIC-8_3.9x4.9mm_P1.27mm, symbol Comparator:LT1011
- added Y1: Crystal, Crystal:Crystal_HC49-U_Vertical, symbol Device:Crystal
- C3: value 200u -> C; footprint (none) -> Capacitor_THT:C_Axial_L3.8mm_D2.6mm_P7.50mm_Horizontal
- D5, D6: footprint (none) -> Diode_SMD:D_MELF-RM10_Universal_Handsoldering
- R1, R2: value 75k -> 4.7k; footprint (none) -> Resistor_THT:R_Axial_DIN0207_L6.3mm_D2.5mm_P10.16mm_Horizontal
- R3: value 58.695k -> R; footprint (none) -> Resistor_THT:R_Axial_DIN0207_L6.3mm_D2.5mm_P10.16mm_Horizontal
- R4: value 91.304k -> R; footprint (none) -> Resistor_THT:R_Axial_DIN0207_L6.3mm_D2.5mm_P10.16mm_Horizontal
- R5: value 1k -> R; footprint (none) -> Resistor_THT:R_Axial_DIN0207_L6.3mm_D2.5mm_P10.16mm_Horizontal
- R6: value 4928 -> R; footprint (none) -> Resistor_THT:R_Axial_DIN0207_L6.3mm_D2.5mm_P10.16mm_Horizontal
- R7: value 2975 -> R; footprint (none) -> Resistor_THT:R_Axial_DIN0207_L6.3mm_D2.5mm_P10.16mm_Horizontal
- R8: value 595 -> R; footprint (none) -> Resistor_THT:R_Axial_DIN0207_L6.3mm_D2.5mm_P10.16mm_Horizontal
- U1, U4, U5, V3: now not fitted; now left out of the parts list
Connections:
- net GND: now also C3.2, R6.1, C1.2, C13.2, C14.2, C5.1, C_G1.1, C_G2.1, ConnProgramator1.1 (Pin_1), J1.3 (Pin_3), R10.1, R16.2, R28.1, R34.2, R36.1, R39.1, R42.1, R43.2, R45.2, R9.2, U11.2, U11.3, U12.2, U13.3 (+), U13.5 (+), U14.3 (+), U15.5 (+), U18.2 (VSS), U19.1 (GND), U3.6 (GND), U7.23 (VSS), U7.35 (VSS), U7.47 (VSS), U7.49 (VSS), U8.1 (GND), U8.2 (+), U9.3 (+); no longer R2.1, R4.2, R7.1, R8.1, U1.2 (Y2), U1.4 (Z), U1.8 (X2), U4.3 (+), U4.4 (V-), U4.5 (+)
- net at D6.1 (K): now also Button2_b1.1 (Pin_1), U17.2
- net at R3.1: now also U14.14 (+)
- net at U1.6 (+VS): now also U1.5 (W)
- net at R7.2: now also C3.1, U2.3 (+)
- net at R8.2: now also U6.6 (-), U6.7
- net at D5.2 (A): now also D6.2 (A), R9.1
- net at U4.2 (-): no longer R6.1
- net at R5.1: now also U2.6 (-), U2.7
- net SCL: now reaches R1.2
- net SCL: now also U18.5 (SCL), U7.42 (PB6)
- net at R5.2: now also C1.1, U6.3 (+); no longer U4.8 (V+)
- net at U4.6 (-): no longer U4.7
- new net: C10.1, C7.2, R14.2, U9.2 (-)
- new net: C10.2, ConnView_Out4.1 (Pin_1), R14.1, U9.1, U9.5 (+)
- new net: C6.1, ConnView_Out2.1 (Pin_1), U6.1, U6.2 (-)
- new net: ConnView_OutLast1.1 (Pin_1), U16.3, U17.3
- new net: C_G2.2, U7.6 (PH1), Y1.1
- new net: Q3.2 (B), R15.1, R20.1
- new net: Button1_b2.1 (Pin_1), R19.2, R20.2, U12.4
- new net: R31.2, R32.1, U13.6 (-)
- new net: ConnView_Modulation1.1 (Pin_1), R24.2, R32.2, U13.7
- new net: C_G1.2, U7.5 (PH0), Y1.2
- new net: C6.2, ConnView_Out3.1 (Pin_1), R10.2, U8.3 (-)
- new net: Q3.3 (C), R27.1
- new net: R27.2, U11.1
- new net: R3.2, R4.2, U14.13 (-)
- new net: Q4.1 (E), Q5.2 (B), R34.1, R35.2, R45.1
- new net: Button1_a1.1 (Pin_1), D1.1 (K)
- new net: D1.2 (A), U9.6 (-), U9.7
- new net: R16.1, U16.1, U17.1
- new net: Button2_b2.1 (Pin_1), D5.1 (K), U16.2
- new net: R22.2, U15.7, U16.4
- new net: Button1_a2.1 (Pin_1), U10.1, U10.2 (-)
- new net: ConnView_Out5.1 (Pin_1), R13.1, R6.2, U10.3 (+), U6.5 (+), U8.7
- new net: Q5.1 (E), R29.1, R43.1
- new net: R29.2, R30.1, U13.2 (-)
- new net: ConnView_Out1.1 (Pin_1), Q1.2 (B), R41.1, R42.2
- new net: C5.2, Q4.2 (B), R18.2, U12.3
- new net: U5.GND, V3.2
- new net: R11.2, R24.1, U14.16
- new net: C7.1, R8.1
- new net: R21.2, U12.1
- new net: Q1.3 (C), R40.1
- new net: R37.1, R38.2, U2.1
- new net: C13.1, R37.2, U2.5 (+)
- new net: U15.1, U15.2 (-), U17.4
- new net: U14.4 (-), U14.5
- new net: R36.2, R38.1, U2.2 (-)
- new net: R17.1, R23.2, U14.9, U15.3 (+)
- new net: Q2.1 (E), R21.1
- new net: Q3.1 (E), R26.1, R28.2
- new net: ConnView_OutInfo1.1 (Pin_1), R11.1, R4.1, U10.6 (-), U10.7
- new net: Q2.2 (B), R19.1
- new net: Button1_b1.1 (Pin_1), R15.2, R18.1, U11.4
- new net: R30.2, R31.1, U13.1
- new net: R17.2, R22.1, U15.6 (-)
- new net: Q1.1 (E), R39.2, R7.1
- new net: Q5.3 (C), R44.2
- new net: U14.10, U14.12
- new net: R25.1, U14.15 (DIODE_BIAS)
- new net 3V3: ConnProgramator1.4 (Pin_4), U19.2 (VO), U7.1 (VBAT), U7.24 (VDD), U7.36 (VDD), U7.48 (VDD), U7.9 (VDDA)
- new net LCD_CS: U3.25 (LCD_CS), U7.19 (PB1)
- new net LCD_DC: U3.22 (LCD_DS), U7.18 (PB0)
- new net MISO: U3.27 (MISO), U7.16 (PA6)
- new net MOSI: U3.26 (MOSI), U7.17 (PA7)
- new net SCLK: U3.28 (SCLK), U7.15 (PA5)
- new net SDA: R2.2, U18.4 (SDA), U7.43 (PB7)
- new net SD_CS: U3.20 (SD_CS), U7.40 (PB4)
- new net SWCLK: ConnProgramator1.2 (Pin_2), U7.37 (PA14)
- new net SWDIO: ConnProgramator1.3 (Pin_3), U7.34 (PA13)
- new net Signal_drwng: U10.5 (+), U18.1 (VOUT)
- new net TP_CS: U3.19 (TP_CS), U7.20 (PB2)
- new net TP_IRQ: U3.18 (TP_IRQ), U7.25 (PB12)
- new net V15: C14.1, J1.1 (Pin_1), Q4.3 (C), R13.2, R25.2, R35.1, R40.2, R41.2, R44.1, U10.8 (V+), U13.8 (V+), U14.11 (V+), U15.8 (V+), U2.8 (V+), U6.8 (V+), U8.8 (V+), U9.8 (V+)
- new net V15m: Button2_a1.1 (Pin_1), Button2_a2.1 (Pin_1), J1.5 (Pin_5), R23.1, U10.4 (V-), U13.4 (V-), U14.6 (V-), U15.4 (V-), U2.4 (V-), U6.4 (V-), U8.4 (V-), U9.4 (V-)
- new net V5: J1.2 (Pin_2), Q2.3 (C), R1.1, R2.1, R26.2, U18.3 (VDD), U19.3 (VI), U3.24 (LCD_BL), U3.5 (+5V)
- new net V5m: J1.4 (Pin_4)
- now unconnected: U1.1 (Y1), U1.7 (X1), U4.1, U5.B10, U5.GND
Other:
- note added: "27pF"
- moved on the sheet: D5, D6
