File: DrawerModeling/DrawerModeling.kicad_sch (KiCad schematic)
At the start: 101 parts, among them J1 Conn_01x05_Pin, Q1 2N3904, Q2 2N3904, Q3 2N3906, Q4 2N3904, Q5 2N3904, U1 AD633JRZ-R7, U10 TL072, U11 TLP222A, U12 TLP222A, U13 TL072, U14 LM13700, U15 TL072, U16 TLP222A, U17 TLP222A, U18 MCP4725xxx-xCH, U19 XC6206PxxxMR, U2 TL072, U4 TL082_Block, U6 TL072, U7 STM32F411CCUx, U8 LT1011, U9 TL072, Y1 Crystal

Commit message: recovery after bad days
Parts:
- removed D5, D6: D, Diode_SMD:D_MELF-RM10_Universal_Handsoldering, symbol Device:D
- removed U7: STM32F411CCUx, Package_DFN_QFN:QFN-48-1EP_7x7mm_P0.5mm_EP5.6x5.6mm, symbol MCU_ST_STM32F4:STM32F411CCUx
- added C2: C, Capacitor_THT:C_Axial_L3.8mm_D2.6mm_P7.50mm_Horizontal, symbol Device:C
- added C_s1, C_s3, C_s4, C_s8: 100n, Capacitor_SMD:C_0603_1608Metric, symbol Device:C
- added C_s5, C_s6: 1u, Capacitor_SMD:C_0603_1608Metric, symbol Device:C
- added C_s7: C, Capacitor_SMD:C_0603_1608Metric, symbol Device:C
- added D5, D6: LED, LED_THT:LED_D5.0mm, symbol Device:LED
- added R33, R46: R, Resistor_THT:R_Axial_DIN0207_L6.3mm_D2.5mm_P10.16mm_Horizontal, symbol Device:R
- added R60: 10k, Resistor_THT:R_Axial_DIN0207_L6.3mm_D2.5mm_P10.16mm_Horizontal, symbol Device:R
- added U20: LT1011, Package_SO:SOIC-8_3.9x4.9mm_P1.27mm, symbol Comparator:LT1011
- added U7: STM32F401CCUx, Package_DFN_QFN:QFN-48-1EP_7x7mm_P0.5mm_EP5.6x5.6mm, symbol MCU_ST_STM32F4:STM32F401CCUx
- added UART1: Conn_01x03_Pin, Connector_PinHeader_2.54mm:PinHeader_1x03_P2.54mm_Vertical, symbol Connector:Conn_01x03_Pin
- added Vw_GND1: Conn_01x01, Connector_Wire:SolderWirePad_1x01_SMD_1.5x3mm, symbol Connector_Generic:Conn_01x01
- D1: value D -> 1N4148; footprint Diode_SMD:D_MELF-RM10_Universal_Handsoldering -> Diode_THT:D_DO-35_SOD27_P7.62mm_Horizontal
- renumbered Button1_a1 to B1_a1, Button1_a2 to B1_a2, Button1_b1 to B1_b1, Button1_b2 to B1_b2, Button2_a1 to B2_a1, Button2_a2 to B2_a2, Button2_b1 to B2_b1, Button2_b2 to B2_b2, ConnView_OutInfo1 to Vw_MC1, ConnView_Modulation1 to Vw_Mdltn1, ConnView_OutLast1 to Vw_Out1, ConnView_Out1 to Vw_PWM1, ConnView_Out2 to Vw_SIN+Cnst1, ConnView_Out3 to Vw_SIN1, ConnView_Out5 to Vw_long1, ConnView_Out4 to Vw_short1
Connections:
- net 3V3: now also C_s1.1, C_s3.1, C_s4.1, C_s6.2, R33.2, U20.8 (V+), U7.1 (VBAT), U7.24 (VDD), U7.36 (VDD), U7.48 (VDD), U7.9 (VREF+)
- net GND: now also C2.2, C_s1.2, C_s3.2, C_s4.2, C_s5.1, C_s6.1, C_s7.1, C_s8.2, R46.1, R60.1, U20.1 (GND), U20.2 (+), U20.4 (V-), U7.23 (VSS), U7.35 (VSS), U7.47 (VSS), U7.49 (VSS), U7.8 (VSSA), UART1.3 (Pin_3), Vw_GND1.1 (Pin_1)
- net LCD_CS: now also U7.19 (PB1)
- net LCD_DC: now also U7.18 (PB0)
- net MISO: now also U7.16 (PA6)
- net MOSI: now also U7.17 (PA7)
- net SCL: now also U7.42 (PB6)
- net SCLK: now also U7.15 (PA5)
- net SDA: now also U7.43 (PB7)
- net SD_CS: now also U7.40 (PB4)
- net SWCLK: now also U7.37 (PA14)
- net SWDIO: now also U7.34 (PA13)
- net TP_CS: now also U7.20 (PB2)
- net TP_IRQ: now also U7.25 (PB12)
- net V15: now also C2.1
- net V5: now also C_s5.2
- net at C_G2.2, Y1.1: now also U7.6 (PH1)
- net at B2_b1.1 (Pin_1), U17.2: now also D6.1 (K)
- net at R9.1: now also D5.2 (A), D6.2 (A)
- net at C_G1.2, Y1.2: now also U7.5 (PH0)
- net at C6.2, R10.2, U8.3 (-)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: now also U20.3 (-)
- net at B2_b2.1 (Pin_1), U16.2: now also D5.1 (K)
- net PWM: now reaches Q1.2 (B), R41.1, R42.2, Vw_PWM1.1 (Pin_1)
- net PWM: now also U7.10 (PA0)
- new net: R60.2, U7.44 (BOOT0)
- new net: R33.1, R46.2, U20.7, U7.13 (PA3)
- new net: C_s7.2, U7.22 (VCAP1)
- new net: C_s8.1, U7.7 (NRST)
- new net RX: U7.31 (PA10), UART1.2 (Pin_2)
- new net TX: U7.30 (PA9), UART1.1 (Pin_1)
Other:
- moved on the sheet: C_G1, C_G2, ConnProgramator1, U19, Y1
