File: DrawerModeling/PowerDrwr/PowerDrwr.kicad_pcb (KiCad board)
At the start: 2 copper layers, 59.5 x 41.5 mm, 23 parts, among them J1 Conn_01x05_Pin, U1 LT1086-ADJ, U2 L7915, U3 LT1086-ADJ, U4 LM337_TO220

Commit message: recovery after bad days
Parts:
- removed the REF** at (28.0, 49.0)
- removed the REF** at (80.5, 49.0)
- removed the REF** at (80.5, 83.5)
- removed the REF** at (28.0, 83.5)
- added B1_a1: Conn_01x01, Connector_Wire:SolderWirePad_1x01_SMD_1.5x3mm, F.Cu at (52.8, 32.6)
- added B1_a2: Conn_01x01, Connector_Wire:SolderWirePad_1x01_SMD_1.5x3mm, F.Cu at (52.9, 69.1)
- added B1_b1: Conn_01x01, Connector_Wire:SolderWirePad_1x01_SMD_1.5x3mm, F.Cu at (56.4, 69.1)
- added B1_b2: Conn_01x01, Connector_Wire:SolderWirePad_1x01_SMD_1.5x3mm, F.Cu at (56.2, 32.6)
- added L1: LED, LED_THT:LED_D5.0mm, F.Cu at (89.3, 36.4)
- added R3: R, Resistor_THT:R_Axial_DIN0207_L6.3mm_D2.5mm_P10.16mm_Horizontal, F.Cu at (83.0, 41.2)
- added REF**: MountingHole_3.2mm_M3, MountingHole:MountingHole_3.2mm_M3, F.Cu at (97.9, 68.0)
- added REF**: MountingHole_3.2mm_M3, MountingHole:MountingHole_3.2mm_M3, F.Cu at (45.5, 33.6)
- added REF**: MountingHole_3.2mm_M3, MountingHole:MountingHole_3.2mm_M3, F.Cu at (97.9, 33.6)
- added REF**: MountingHole_3.2mm_M3, MountingHole:MountingHole_3.2mm_M3, F.Cu at (45.5, 68.0)
- moved C2 23.7 mm to (52.0, 50.1)
- moved C1 23.3 mm to (92.5, 45.4)
- moved C4 23.3 mm to (73.5, 43.9)
- moved C5 23.3 mm to (73.5, 51.1)
- moved C8 23.3 mm to (86.5, 45.1)
- moved C9 23.3 mm to (93.0, 60.6)
- moved J1 23.3 mm to (98.5, 46.5)
- moved R12 23.3 mm to (87.0, 67.7)
- moved R133 23.3 mm to (81.5, 62.2)
- moved U3 23.3 mm to (76.0, 36.1)
- moved U4 23.3 mm to (73.5, 59.5)
- moved C12 23.3 mm to (50.5, 58.6)
- moved R2 23.3 mm to (62.5, 45.0)
- moved VCC1 23.3 mm to (44.0, 44.6)
- moved VEE1 23.3 mm to (44.0, 60.1)
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- renumbered VCC to VCC1, VEE to VEE1, GND to VSS1
Connections:
- C12 pad 2: Net-(U2-VI) -> Net-(B1_b1-Pin_1)
- C2 pad 1: Net-(U1-VI) -> Net-(B1_b2-Pin_1)
- U1 pad 3: Net-(U1-VI) -> Net-(B1_b2-Pin_1)
- U2 pad 2: Net-(U2-VI) -> Net-(B1_b1-Pin_1)
- VCC1 pad 1: Net-(U1-VI) -> Net-(B1_a1-Pin_1)
- VEE1 pad 1: Net-(U2-VI) -> Net-(B1_a2-Pin_1)
Routing:
- net Net-(B1_b1-Pin_1): track 0.00 -> 23.2 mm
- net /V15: track 93.4 -> 70.4 mm
- net GND: track 89.9 -> 112.3 mm
- net Net-(B1_b2-Pin_1): track 0.00 -> 21.3 mm
- net Net-(U2-VI): track 19.3 -> 0.00 mm
- net Net-(B1_a1-Pin_1): track 0.00 -> 17.4 mm
- net Net-(U1-VI): track 15.6 -> 0.00 mm
- net Net-(B1_a2-Pin_1): track 0.00 -> 14.4 mm
- net Net-(L1-K): track 0.00 -> 6.49 mm
- net /V5: track 38.9 -> 44.7 mm
- net /V15m: track 65.9 -> 70.4 mm
- net Net-(U1-ADJ): track 14.2 -> 11.5 mm
- net /V5m: track 36.2 -> 36.9 mm
Other:
- board text added: "OscilloscopeDrawer"
- board text added: "R1"
- board text added: "U4"
