File: DrawerModeling/PowerDrwr/PowerDrwr.kicad_sch (KiCad schematic)
At the start: 19 parts, among them J1 Conn_01x05_Pin, U1 LT1086-ADJ, U2 L7915, U3 LT1086-ADJ, U4 LM337_TO220

Commit message: recovery after bad days
Parts:
- added B1_a1, B1_a2, B1_b1, B1_b2: Conn_01x01, Connector_Wire:SolderWirePad_1x01_SMD_1.5x3mm, symbol Connector_Generic:Conn_01x01
- added L1: LED, LED_THT:LED_D5.0mm, symbol Device:LED
- added R3: R, Resistor_THT:R_Axial_DIN0207_L6.3mm_D2.5mm_P10.16mm_Horizontal, symbol Device:R
- renumbered GND_conn1 to VSS1
Connections:
- net GND: now also R3.1
- net V5: now also L1.2 (A)
- net at C2.1, U1.3 (VI): now also B1_b2.1 (Pin_1); no longer VCC1.1 (Pin_1)
- net at C12.2, U2.2 (VI): now also B1_b1.1 (Pin_1); no longer VEE1.1 (Pin_1)
- new net: B1_a1.1 (Pin_1), VCC1.1 (Pin_1)
- new net: B1_a2.1 (Pin_1), VEE1.1 (Pin_1)
- new net: L1.1 (K), R3.2
Other:
- moved on the sheet: J1, VCC1, VEE1
